File: boards/hellen121vag-a/kicad6/hellen121vag.kicad_pcb (KiCad board)
At the start: 2 copper layers, 164 x 118 mm, 115 parts, among them J1 USB_B_Mini, J10 AudioJack3_SwitchTR, J2 Conn_01x01, J3 Conn_01x01, J4 Conn_01x01, J5 Conn_01x01, J6 Conn_01x01, J7 Conn_01x04, J8 Conn_01x06, J9 Conn_01x04, M1 Module-can-0.1, M10 Module-can-0.1, M11 Module-vr-0.1, M12 Module-dinput4-0.1, M2 Module-power5-0.2, M3 Module-mcu-0.1, M4 Module-input-0.1, M5 Module-knock-0.1, M6 Module-output-0.1, M7 Module-ign8-0.1, M8 Module-power12-0.1, M9 Module-wbo-0.1, P1 368255-2, U1 L6205PD, U2 LPS25HB, U3 MCP6002-xSN

Commit message: Upd replace
Parts:
- moved J10 3.80 mm to (144.4, 6.17)
- moved J1 1.82 mm to (128.8, 7.20)
Routing:
- net GND: track 13.5 -> 8.38 mm

Commit message: Upd h1
Parts:
- J10: value AudioJack3_SwitchTR -> AudioJack_THR
Changed lines of the file:
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@@
       (xy -2.15345 -5.80914)) (layer "F.Fab") (width 0.01) (fill solid))
     (pad "1" smd rect (at -5.715 6.6) (size 0.8 2.2) (layers "F.Cu" "F.Paste" "F.Mask")
-      (net 8 "GND") (pinfunction "GND@1"))
+      (net 8 "GND") (pinfunction "GND@1") (pintype "power_in"))
     (pad "2" smd rect (at -4.445 6.6) (size 0.8 2.2) (layers "F.Cu" "F.Paste" "F.Mask")
-      (net 232 "+12V_RAW") (pinfunction "VSA"))
+      (net 232 "+12V_RAW") (pinfunction "VSA") (pintype "power_in"))
     (pad "3" smd rect (at -3.175 6.6) (size 0.8 2.2) (layers "F.Cu" "F.Paste" "F.Mask")
-      (net 279 "/+ETB_OUT") (pinfunction "OUT2A"))
+      (net 279 "/+ETB_OUT") (pinfunction "OUT2A") (pintype "output"))
     (pad "4" smd rect (at -1.905 6.6) (size 0.8 2.2) (layers "F.Cu" "F.Paste" "F.Mask")
-      (net 180 "Net-(C4-Pad1)") (pinfunction "VCP"))
+      (net 180 "Net-(C4-Pad1)") (pinfunction "VCP") (pintype "passive"))
     (pad "5" smd rect (at -0.635 6.6) (size 0.8 2.2) (layers "F.Cu" "F.Paste" "F.Mask")
-      (net 181 "Net-(C5-Pad2)") (pinfunction "ENA"))
+      (net 181 "Net-(C5-Pad2)") (pinfunction "ENA") (pintype "bidirectional"))
     (pad "6" smd rect (at 0.635 6.6) (size 0.8 2.2) (layers "F.Cu" "F.Paste" "F.Mask")
-      (net 273 "/-ETB") (pinfunction "IN1A"))
+      (net 273 "/-ETB") (pinfunction "IN1A") (pintype "input"))
     (pad "7" smd rect (at 1.905 6.6) (size 0.8 2.2) (layers "F.Cu" "F.Paste" "F.Mask")
-      (net 272 "/+ETB") (pinfunction "IN2A"))
+      (net 272 "/+ETB") (pinfunction "IN2A") (pintype "input"))
     (pad "8" smd rect (at 3.175 6.6) (size 0.8 2.2) (layers "F.Cu" "F.Paste" "F.Mask")
-      (net 8 "GND") (pinfunction "SENSEA"))
+      (net 8 "GND") (pinfunction "SENSEA") (pintype "power_in"))
     (pad "9" smd rect (at 4.445 6.6) (size 0.8 2.2) (layers "F.Cu" "F.Paste" "F.Mask")
-      (net 280 "/-ETB_OUT") (pinfunction "OUT1A"))
+      (net 280 "/-ETB_OUT") (pinfunction "OUT1A") (pintype "output"))
     (pad "10" smd rect (at 5.715 6.6) (size 0.8 2.2) (layers "F.Cu" "F.Paste" "F.Mask")
-      (net 8 "GND") (pinfunction "GND@2"))
+      (net 8 "GND") (pinfunction "GND@2") (pintype "power_in"))
     (pad "11" smd rect (at 5.715 -6.6) (size 0.8 2.2) (layers "F.Cu" "F.Paste" "F.Mask")
-      (net 8 "GND") (pinfunction "GND@3"))
+      (net 8 "GND") (pinfunction "GND@3") (pintype "power_in"))
     (pad "12" smd rect (at 4.445 -6.6) (size 0.8 2.2) (layers "F.Cu" "F.Paste" "F.Mask")
-      (net 280 "/-ETB_OUT") (pinfunction "OUT1B"))
+      (net 280 "/-ETB_OUT") (pinfunction "OUT1B") (pintype "output"))
     (pad "13" smd rect (at 3.175 -6.6) (size 0.8 2.2) (layers "F.Cu" "F.Paste" "F.Mask")
-      (net 8 "GND") (pinfunction "SENSEB"))
+      (net 8 "GND") (pinfunction "SENSEB") (pintype "power_in"))
     (pad "14" smd rect (at 1.905 -6.6) (size 0.8 2.2) (layers "F.Cu" "F.Paste" "F.Mask")
-      (net 273 "/-ETB") (pinfunction "IN1B"))
+      (net 273 "/-ETB") (pinfunction "IN1B") (pintype "input"))
     (pad "15" smd rect (at 0.635 -6.6) (size 0.8 2.2) (layers "F.Cu" "F.Paste" "F.Mask")
-      (net 272 "/+ETB") (pinfunction "IN2B"))
+      (net 272 "/+ETB") (pinfunction "IN2B") (pintype "input"))
     (pad "16" smd rect (at -0.635 -6.6) (size 0.8 2.2) (layers "F.Cu" "F.Paste" "F.Mask")
-      (net 181 "Net-(C5-Pad2)") (pinfunction "ENB"))
+      (net 181 "Net-(C5-Pad2)") (pinfunction "ENB") (pintype "bidirectional"))
     (pad "17" smd rect (at -1.905 -6.6) (size 0.8 2.2) (layers "F.Cu" "F.Paste" "F.Mask")
-      (net 83 "Net-(C3-Pad1)") (pinfunction "VBOOT"))
+      (net 83 "Net-(C3-Pad1)") (pinfunction "VBOOT") (pintype "passive"))
     (pad "18" smd rect (at -3.175 -6.6) (size 0.8 2.2) (layers "F.Cu" "F.Paste" "F.Mask")
-      (net 279 "/+ETB_OUT") (pinfunction "OUT2B"))
+      (net 279 "/+ETB_OUT") (pinfunction "OUT2B") (pintype "output"))
     (pad "19" smd rect (at -4.445 -6.6) (size 0.8 2.2) (layers "F.Cu" "F.Paste" "F.Mask")
-      (net 232 "+12V_RAW") (pinfunction "VSB"))
+      (net 232 "+12V_RAW") (pinfunction "VSB") (pintype "power_in"))
     (pad "20" smd rect (at -5.715 -6.6) (size 0.8 2.2) (layers "F.Cu" "F.Paste" "F.Mask")
-      (net 8 "GND") (pinfunction "GND@4"))
+      (net 8 "GND") (pinfunction "GND@4") (pintype "power_in"))
     (pad "SLUG1" smd rect (at -7.112 0) (size 2.032 5.08) (layers "F.Cu" "F.Paste" "F.Mask")
-      (net 8 "GND") (pinfunction "SLUG@1") (zone_connect 2))
+      (net 8 "GND") (pinfunction "SLUG@1") (pintype "power_in") (zone_connect 2))
     (pad "SLUG2" smd rect (at 0 0) (size 11.43 7.62) (layers "F.Cu" "F.Paste" "F.Mask")
-      (net 8 "GND") (pinfunction "SLUG@2") (zone_connect 2))
+      (net 8 "GND") (pinfunction "SLUG@2") (pintype "power_in") (zone_connect 2))
     (pad "SLUG3" smd rect (at 7.112 0) (size 2.032 5.08) (layers "F.Cu" "F.Paste" "F.Mask")
-      (net 8 "GND") (pinfunction "SLUG@3") (zone_connect 2))
+      (net 8 "GND") (pinfunction "SLUG@3") (pintype "power_in") (zone_connect 2))
   )
   (footprint "hellen-one-can-0.1:can" (layer "F.Cu")
@@
       (effects (font (size 1 1) (thickness 0.15)))
     )
-    (fp_text value "AudioJack3_SwitchTR" (at 0.1 14.05 90) (layer "F.Fab")
+    (fp_text value "AudioJack_THR" (at 0.1 14.05 90) (layer "F.Fab")
       (effects (font (size 1 1) (thickness 0.15)))
     )
@@
     (fp_line (start 3.8 -9) (end 3.8 -5) (layer "F.Fab") (width 0.1))
     (pad "R" thru_hole oval (at 1.9 4.3 315) (size 3 2.4) (drill 2) (layers *.Cu *.Mask)
-      (net 302 "unconnected-(J10-PadR)"))
+      (net 302 "unconnected-(J10-PadR)") (pintype "passive+no_connect"))
     (pad "RN" thru_hole oval (at -0.3 2.4 315) (size 3 2.4) (drill 2) (layers *.Cu *.Mask)
-      (net 301 "unconnected-(J10-PadRN)"))
+      (net 301 "unconnected-(J10-PadRN)") (pintype "passive+no_connect"))
     (pad "S" thru_hole oval (at -0.3 -3.8 315) (size 3 2.4) (drill 2) (layers *.Cu *.Mask)
-      (net 8 "GND"))
+      (net 8 "GND") (pintype "passive"))
     (pad "T" thru_hole oval (at 1.9 -1.3 315) (size 3 2.4) (drill 2) (layers *.Cu *.Mask)
-      (net 299 "Net-(C17-Pad1)"))
+      (net 299 "Net-(C17-Pad1)") (pintype "passive"))
     (pad "TN" thru_hole oval (at -0.3 8 315) (size 3 2.4) (drill 2) (layers *.Cu *.Mask)
-      (net 300 "unconnected-(J10-PadTN)"))
+      (net 300 "unconnected-(J10-PadTN)") (pintype "passive+no_connect"))
     (model "${KICAD6_3DMODEL_DIR}/Connector_Audio.3dshapes/Jack_3.5mm_CUI_SJ1-3535NG_Horizontal.wrl"
       (offset (xyz -0.1 3.8 0))
@@
     (fp_line (start -3.6 1.775) (end -2.3 1.775) (layer "F.Fab") (width 0.15))
     (pad "1" thru_hole rect (at -1.6 0.875) (locked) (size 1.1 1.1) (drill 0.7) (layers *.Cu *.Mask)
-      (net 12 "/VBUS") (pinfunction "VBUS"))
+      (net 12 "/VBUS") (pinfunction "VBUS") (pintype "power_out"))
     (pad "2" thru_hole circle (at -0.8 -0.875) (locked) (size 1.1 1.1) (drill 0.7) (layers *.Cu *.Mask)
-      (net 15 "/USBM") (pinfunction "D-"))
+      (net 15 "/USBM") (pinfunction "D-") (pintype "passive"))
     (pad "3" thru_hole circle (at 0 0.875) (locked) (size 1.1 1.1) (drill 0.7) (layers *.Cu *.Mask)
-      (net 13 "/USBP") (pinfunction "D+"))
+      (net 13 "/USBP") (pinfunction "D+") (pintype "passive"))
     (pad "4" thru_hole circle (at 0.8 -0.875) (locked) (size 1.1 1.1) (drill 0.7) (layers *.Cu *.Mask)
-      (net 231 "unconnected-(J1-Pad4)") (pinfunction "ID"))
+      (net 231 "unconnected-(J1-Pad4)") (pinfunction "ID") (pintype "passive+no_connect"))
     (pad "5" thru_hole circle (at 1.6 0.875) (locked) (size 1.1 1.1) (drill 0.7) (layers *.Cu *.Mask)
-      (net 8 "GND") (pinfunction "GND"))
+      (net 8 "GND") (pinfunction "GND") (pintype "power_out"))
     (pad "6" thru_hole oval (at 3.65 0) (locked) (size 1.1 2.4) (drill oval 0.7 2) (layers *.Cu *.Mask)
-      (net 230 "unconnected-(J1-Pad6)") (pinfunction "Shield"))
+      (net 230 "unconnected-(J1-Pad6)") (pinfunction "Shield") (pintype "passive+no_connect"))
     (pad "6" thru_hole oval (at -3.65 0) (locked) (size 1.1 2.4) (drill oval 0.7 2) (layers *.Cu *.Mask)
-      (net 230 "unconnected-(J1-Pad6)") (pinfunction "Shield"))
+      (net 230 "unconnected-(J1-Pad6)") (pinfunction "Shield") (pintype "passive+no_connect"))
     (model "${KICAD6_3DMODEL_DIR}/Connector_USB.3dshapes/USB_Mini-B_Tensility_54-00023_Vertical.wrl"
       (offset (xyz -1.6 -0.875 0))

Commit message: Fabrication outputs
Parts:
- added R20: 1.6k, hellen-one-common:R0603, F.Cu at (54.8, 27.0)
- added R21: 750, hellen-one-common:R0603, F.Cu at (54.8, 29.5)
- R16: value 4.7k -> 5.1k; footprint hellen-one-common:R0603-4 -> hellen-one-common:R0603
- R17: value 470 -> 5.1k; footprint hellen-one-common:R0603-4 -> hellen-one-common:R0603
- moved R17 10.7 mm to (54.8, 17.5), turned to 180 degrees
- moved R16 1.28 mm to (54.8, 15.0), turned to 180 degrees
Connections:
- R16 pad 1: GND -> Net-(D3-Pad2)
- R17 pad 1: GND -> Net-(D5-Pad2)
Routing:
- net Net-(D7-Pad2): track 5.59 -> 3.91 mm
