File: hellen121vag.kicad_sch (KiCad schematic)
At the start: 117 parts, among them J1 USB_B_Mini, J10 AudioJack_THR, J2 Conn_01x01, J3 Conn_01x01, J4 Conn_01x01, J5 Conn_01x01, J6 Conn_01x01, J7 Conn_01x04, J8 Conn_01x06, J9 Conn_01x04, M1 Module-can-0.1, M10 Module-can-0.1, M11 Module-vr-0.1, M12 Module-dinput4-0.1, M2 Module-power5-0.2, M3 Module-mcu-0.1, M4 Module-input-0.1, M5 Module-knock-0.1, M6 Module-output-0.1, M7 Module-ign8-0.1, M8 Module-power12-0.1, M9 Module-wbo-0.1, P1 368255-2, U1 L6205PD, U2 LPS25HB, U3 MCP6002-xSN

Commit message: Upd sch: #25, #27, #28, #33, #34, #36, #37 and new versions of modules
Parts:
- removed M3: Module-mcu-0.1, hellen-one-mcu-0.1:mcu, symbol hellen-one-mcu-0.1:Module-mcu-0.1
- removed M6: Module-output-0.1, hellen-one-output-0.1:output, symbol hellen-one-output-0.1:Module-output-0.1
- removed M8: Module-power12-0.1, hellen-one-power12-0.1:power12, symbol hellen-one-power12-0.1:Module-power12-0.1
- added C18: 100n, hellen-one-common:C0603, symbol hellen-one-common:Cap
- added D10, D11, D12: 1N4148WS, hellen-one-common:SOD-323, symbol hellen-one-common:1N4148WS
- added G4: DISCLAIMER, rusefi_lib:Off_Road_Disclaimer, symbol Off_Road_Disclaimer:Disclaimer
- added G7: LOGO, rusefi_lib:LOGO, symbol logo:LOGO
- added J11: Conn_01x06, Connector_PinHeader_2.54mm:PinHeader_1x06_P2.54mm_Vertical, symbol Connector_Generic:Conn_01x06
- added M13: Module-sd-0.1, hellen-one-sd-0.1:sd, symbol hellen-one-sd-0.1:Module-sd-0.1
- added M3: Module-mcu-0.2, hellen-one-mcu-0.2:mcu, symbol hellen-one-mcu-0.2:Module-mcu-0.2
- added M6, M?: Module-output-0.2, hellen-one-output-0.2:output, symbol hellen-one-output-0.2:Module-output-0.2
- added M8: Module-power12-0.2, hellen-one-power12-0.2:power12, symbol hellen-one-power12-0.2:Module-power12-0.2
- added P2, P3, P4: Pad, hellen-one-common:PAD-TH, symbol hellen-one-common:Pad
- added R22: 10k, hellen-one-common:R0603, symbol hellen-one-common:Res
- added U4: LIS2DW12TR, hellen-one-common:LGA-12_2x2mm_P0.5mm, symbol hellen-one-common:LIS2DW12TR
- R3, R8: LCSC C17477 -> (none); MyComment (none) -> DNP
Connections:
- net +12V: now also M8.V1 (V12); no longer D5.1 (K), D8.1 (A)
- net +12V_PROT: now also D10.1 (K), D11.1 (K), D12.1 (K), M?.W5 (V12P)
- net +12V_RAW: now also D5.1 (K), D8.1 (A), M8.E2 (V12_RAW), M?.S11 (V12_RAW)
- net +3V3: now also C18.2, J11.1 (Pin_1), M13.V1 (V33), M6.N16 (V33), U4.10 (Vdd_IO), U4.9 (Vdd)
- net +5V: now also M6.S1 (V5), M8.E1 (V5), M?.W14 (V5)
- net +5VA: now also M6.S33 (V5A)
- net +ETB: now also M3.E14 (OUT_PWM2)
- net -ETB: now also M3.E15 (OUT_PWM3)
- net A1: now also M3.S30 (IN_O2S2)
- net A2: now also M3.S22 (IN_MAP3)
- net A3: now also M3.S26 (IN_AUX3)
- net A4: now also M3.S23 (IN_RES3)
- net AFR: now also M3.S16 (IN_O2S)
- net BOOT0: now also M6.N28 (BOOT0)
- net CAM1: now also M3.S15 (IN_CAM), P3.1 (Pin_1)
- net CAM2: now also M3.S27 (IN_AUX4), P4.1 (Pin_1)
- net CAN_RX: now also M3.N2 (CAN_RX)
- net CAN_TX: now also M3.N3 (CAN_TX)
- net CAN_VIO: now also M3.N1 (CAN_VIO)
- net CLT: now also M3.S18 (IN_CLT)
- net CRANK: now also M3.S13 (IN_CRANK), P2.1 (Pin_1)
- net D1: now also M3.S3 (IN_D1)
- net D2: now also M3.S4 (IN_D2)
- net D3: now also M3.S5 (IN_D3)
- net D4: now also M3.S6 (IN_D4)
- net ETB_EN: now also M3.E13 (OUT_IO12), R22.1
- net FUEL_CONSUM: now also M3.E19 (OUT_PWM7), M6.W22 (PP2)
- net GND: now also C18.1, J11.6 (Pin_6), M13.G (GND), M13.V2 (GND), M13.V3 (GND), M6.S2 (GND), M8.S1 (GND), M?.G (GND), M?.S3 (GND), R22.2, U4.6 (GND), U4.7 (RES), U4.8 (GND)
- net GNDA: now also M6.S32 (GNDA)
- net IAT: now also M3.S19 (IN_IAT)
- net IDLE: now also M3.E18 (OUT_PWM6), M6.W38 (LOW3_DUAL)
- net IGN1: now also M3.W1 (OUT_IGN1)
- net IGN2: now also M3.W2 (OUT_IGN2)
- net IGN3: now also M3.W3 (OUT_IGN3)
- net IGN4: now also M3.W4 (OUT_IGN4)
- net IGN5: now also M3.W5 (OUT_IGN5)
- net IGN6: now also M3.W6 (OUT_IGN6)
- net IGN7: now also M3.W7 (OUT_IGN7)
- net IGN8: now also M3.W8 (OUT_IGN8)
- net IGN_V33: now also M6.W10 (IGN_V33)
- net IGN_V5: now also M6.W9 (IGN_V5)
- net INJ1: now also M3.E25 (OUT_INJ1), M6.W24 (INJ1)
- net INJ2: now also M3.E26 (OUT_INJ2), M6.W23 (INJ2)
- net INJ3: now also M3.E29 (OUT_INJ3), M6.W20 (INJ3)
- net INJ4: now also M3.E30 (OUT_INJ4), M6.W19 (INJ4)
- net INJ5: now also M3.E31 (OUT_INJ5), M6.W18 (INJ5)
- net INJ6: now also M3.E32 (OUT_INJ6), M6.W17 (INJ6)
- net INJ7: now also M3.E33 (OUT_INJ7), M6.W16 (INJ7)
- net INJ8: now also M3.E34 (OUT_INJ8), M6.W15 (INJ8)
- net IN_VIGN: now also R8.1, M8.V3 (IN_VIGN); no longer R8.2
- net IO1: now also M6.N12 (IO1); no longer J9.4 (Pin_4)
- net IO2: now also M6.N13 (IO2); no longer J9.3 (Pin_3)
- net IO3: now also M6.N14 (IO3); no longer J9.2 (Pin_2)
- net IO4: now also M6.N15 (IO4); no longer J9.1 (Pin_1)
- net KNOCK1: now also M3.S12 (IN_KNOCK)
- net MAF: now also M3.S20 (IN_MAP1)
- net MAP2: now also M3.S21 (IN_MAP2)
- net NRESET: now also M6.N24 (nReset)
- net OUT1: now also M3.E7 (OUT_IO5), M6.W39 (LOW7_HIGH1)
- net OUT2: now also M3.E9 (OUT_IO6), M6.W37 (LOW8_HIGH2)
- net OUT3: now also M3.E28 (OUT_PWM8), M6.W21 (LOW1)
- net OUT_FUEL_CONSUM: now also M6.S6 (OUT_PP2)
- net OUT_IDLE: now also D12.2 (A), M6.S7 (OUT_LOW3_DUAL)
- net OUT_INJ1: now also M6.S18 (OUT_INJ1)
- net OUT_INJ2: now also M6.S16 (OUT_INJ2)
- net OUT_INJ3: now also M6.S17 (OUT_INJ3)
- net OUT_INJ4: now also M6.W7 (OUT_INJ4)
- net OUT_INJ5: now also M6.W10 (OUT_INJ5)
- net OUT_INJ6: now also M6.S15 (OUT_INJ6)
- net OUT_INJ7: now also M6.W12 (OUT_INJ7)
- net OUT_INJ8: now also M6.W11 (OUT_INJ8)
- net OUT_TACH: now also M6.W6 (OUT_PP1)
- net OUT_VVT1_1: now also M6.S13 (OUT_LOW12), M6.S14 (OUT_LOW9)
- net OUT_VVT1_2: now also M6.W1 (OUT_LOW2), M6.W2 (OUT_LOW10)
- net OUT_VVT2_B1: now also D11.2 (A), M6.S5 (OUT_SOLENOID_B2)
- net OUT_VVT2_B2: now also D10.2 (A), M6.S4 (OUT_SOLENOID_B1)
- net OUT_WASTEGATE: now also M6.W4 (OUT_LOW4_DUAL)
- net PPS1: now also M3.S29 (IN_PPS)
- net PPS2: now also M3.S25 (IN_AUX2)
- net RES1: now also M3.S28 (IN_RES1)
- net RES2: now also M3.S31 (IN_RES2)
- net TACH: now also M3.E27 (OUT_PWM1), M6.W28 (PP1)
- net TPS1: now also M3.S17 (IN_TPS)
- net TPS2: now also M3.S24 (IN_AUX1)
- net USBM: now also M3.N31 (USB1M)
- net USBP: now also M3.N30 (USB1P)
- net V12_PERM: now also M8.V4 (V12_PERM)
- net VBAT: now also M6.N17 (VBAT), M8.V2 (VBAT)
- net VBUS: now also M3.N29 (VBUS)
- net VIGN: now also M3.S7 (VIGN), M8.V5 (VIGN)
- net VSS: now also M3.S14 (IN_VSS)
- net VVT1_1: now also M3.E10 (OUT_IO10), M6.W27 (LOW9), M6.W36 (LOW12)
- net VVT1_2: now also M3.E21 (OUT_IO7), M6.W26 (LOW10), M6.W29 (LOW2)
- net VVT2_B1: now also M3.E17 (OUT_PWM5), M6.W30 (SOLENOID_B2)
- net VVT2_B2: now also M3.E16 (OUT_PWM4), M6.W31 (SOLENOID_B1)
- net WASTEGATE: now also M3.E12 (OUT_IO2), M6.W34 (LOW4_DUAL)
- net at P1.21, R2.1: now also R8.2; no longer R8.1
- net at P1.23: now also R3.2; no longer R3.1
- net at VOUT2.1 (Pin_1): now also M6.S12 (OUT_LOW8_PULLUP)
- net at VOUT3.1 (Pin_1): now also M6.S8 (OUT_LOW1)
- net at R19.2, U2.4 (SDA/MOSI): now also M3.N18 (I2C_SDA)
- net at R18.2, U2.2 (SCL/SCLK): now also M3.N19 (I2C_SCL)
- net at VOUT1.1 (Pin_1): now also M6.W9 (OUT_LOW7_PULLUP)
- net OUT_CE renamed OUT_CHECK_ENGINE
- net OUT_CHECK_ENGINE: now also M6.W3 (OUT_LOW6_DIODE)
- net OUT_MAIN renamed OUT_MAIN_RELAY
- net OUT_MAIN_RELAY: now also R3.1, M6.W13 (OUT_LOW5_MAIN); no longer R3.2
- net OUT_PUMP renamed OUT_FUEL_PUMP_RELAY
- net OUT_FUEL_PUMP_RELAY: now also M6.S10 (OUT_LOW11)
- net SPI2_CS renamed RX2
- net RX2: now also M3.N7 (UART2_RX)
- net SPI2_MISO renamed RX1
- net RX1: now also M3.N5 (UART1_RX)
- net SPI2_MOSI renamed TX2
- net TX2: now also M3.N6 (UART2_TX)
- net SPI2_SCK renamed TX1
- net TX1: now also M3.N4 (UART1_TX)
- new net CHECK_ENGINE: M3.E22 (OUT_IO8), M6.W25 (LOW6_DIODE)
- new net FUEL_PUMP_RELAY: M3.E8 (OUT_IO1), M6.W35 (LOW11)
- new net MAIN_RELAY: M3.E6 (OUT_IO3), M6.W40 (LOW5_MAIN)
- new net SD_CS: J11.2 (Pin_2), M13.V4 (SD_CS), M3.N23 (SPI2_CS)
- new net SD_MISO: J11.5 (Pin_5), M13.V7 (SD_MISO), M3.N21 (SPI2_MISO)
- new net SD_MOSI: J11.3 (Pin_3), M13.V5 (SD_MOSI), M3.N22 (SPI2_MOSI)
- new net SD_SCK: J11.4 (Pin_4), M13.V6 (SD_SCK), M3.N20 (SPI2_SCK)
- new net SPI1_CS: M3.E4 (SPI1_CS1), U4.2 (~CS)
- new net SPI1_MISO: M3.E2 (SPI1_MISO), U4.3 (SA0/SDO)
- new net SPI1_MOSI: M3.E3 (SPI1_MOSI), U4.4 (SDA/SDI)
- new net SPI1_SCK: M3.E1 (SPI1_SCK), U4.1 (SCL/SPC)
- new net SPI3_CS: J9.4 (Pin_4), M3.N8 (SPI3_CS)
- new net SPI3_MISO: J9.2 (Pin_2), M3.N10 (SPI3_MISO)
- new net SPI3_MOSI: J9.1 (Pin_1), M3.N11 (SPI3_MOSI)
- new net SPI3_SCK: J9.3 (Pin_3), M3.N9 (SPI3_SCK)
- no-connect marks 71 -> 62
Other:
- note added: "Accelerometer"
- note added: "Baro"
- moved on the sheet: R18, R19

Commit message: #40, #43
Parts:
- removed unit 4 of M6
- added unit 4 of M3
- gave numbers to parts that had none: 1
Connections:
- net +3V3: now also M3.N16 (V33)
- net +5V: now also M3.S1 (V5)
- net +5VA: now also R6.2, R7.2, M3.S33 (V5A)
- net BOOT0: now also M3.N28 (BOOT0)
- net GND: now also M3.S2 (GND)
- net GNDA: now also M3.S32 (GNDA); no longer R6.2, R7.2
- net IGN_V33: now also M3.W10 (IGN_V33)
- net IGN_V5: now also M3.W9 (IGN_V5)
- net IO1: now also M3.N12 (IO1)
- net IO2: now also M3.N13 (IO2)
- net IO3: now also M3.N14 (IO3)
- net IO4: now also M3.N15 (IO4)
- net NRESET: now also M3.N24 (nReset)
- net VBAT: now also M3.N17 (VBAT)
