File: hellen121vag.kicad_sch (KiCad schematic)
At the start: 128 parts, among them J1 USB_B_Mini, J10 AudioJack_THR, J2 Conn_01x01, J3 Conn_01x01, J4 Conn_01x01, J5 Conn_01x01, J6 Conn_01x01, J7 Conn_01x08, J8 Conn_01x06, M1 Module-can-0.1, M10 Module-can-0.1, M11 Module-vr-discrete-0.1, M2 Module-power5-0.2, M3 Module-mcu-0.7, M4 Module-input-0.1, M5 Module-knock-0.1, M6 Module-output-0.3, M7 Module-ign8-0.2, M8 Module-power12-0.2, M9 Module-wbo-0.3, P1 368255-2, P10 Pad, P11 Pad, P12 Pad, P13 Pad, P14 Pad, P15 Pad, P16 Pad, P17 Pad, P2 Pad, P20 Pad, P28 Pad, P3 Pad, P4 Pad, P40 Pad, P41 Pad, P43 Pad, P44 Pad, P45 Pad, P46 Pad, P48 Pad, P49 Pad, P5 Pad, P56 Pad, P6 Pad, P61 Pad, P63 Pad, P64 Pad, P66 Pad, P67 Pad, P68 Pad, P69 Pad, P7 Pad, P74 Pad, P8 Pad, P80 Pad, P9 Pad, U1 L6205PD, U2 LPS25HB, U3 MCP6002-xSN, U4 TLS115_SOIC, U5 TLS115_SON

Commit message: update schematics to mega, also knock & power #90
Parts:
- removed C15, C6: 100n, hellen-one-common:C0603, symbol hellen-one-common:Cap
- removed C18, C19: 1u, hellen-one-common:C0603, symbol hellen-one-common:Cap
- removed M1, M10: Module-can-0.1, hellen-one-can-0.1:can, symbol hellen-one-can-0.1:Module-can-0.1
- removed M11: Module-vr-discrete-0.1, hellen-one-vr-discrete-0.1:vr-discrete, symbol vr-discrete:Module-vr-discrete-0.1
- removed M2: Module-power5-0.2, hellen-one-power5-0.2:power5, symbol hellen-one-power5-0.2:Module-power5-0.2
- removed M3: Module-mcu-0.7, hellen-one-mcu-0.7:mcu, symbol hellen-one-mcu-0.7:Module-mcu-0.7
- removed unit 1 of M4
- removed unit 3 of M4
- removed unit 2 of M4
- removed M5: Module-knock-0.1, hellen-one-knock-0.1:knock, symbol hellen-one-knock-0.1:Module-knock-0.1
- removed M8: Module-power12-0.2, hellen-one-power12-0.2:power12, symbol hellen-one-power12-0.2:Module-power12-0.2
- removed M9: Module-wbo-0.3, hellen-one-wbo-0.3:wbo, symbol hellen-one-wbo-0.3:Module-wbo-0.3
- removed R18, R19: 4.7k, hellen-one-common:R0603, symbol hellen-one-common:Res
- removed S1, S2: Button_SPST, hellen-one-common:SMD-2_2.9x3.9x1.7, symbol hellen-one-common:Button_SPST
- removed U2: LPS25HB, Package_LGA:ST_HLGA-10_2.5x2.5mm_P0.6mm_LayoutBorder3x2y, symbol Sensor_Pressure:LPS25HB
- removed U4: TLS115_SOIC, kicad6-libraries:PG-DSO-8-43_VIA, symbol hellen-one-common:TLS115
- removed U5: TLS115_SON, Package_SON:HVSON-8-1EP_3x3mm_P0.65mm_EP1.6x2.4mm, symbol hellen-one-common:TLS115
- added M11: Module-vr-discrete-0.4, hellen-one-vr-discrete-0.4:vr-discrete, symbol vr-discrete-0.4:Module-vr-discrete-0.4
- added M3: mega-mcu144-0.1, hellen-one-mega-mcu144-0.1:mega-mcu144, symbol mega-mcu144-0.1:mega-mcu144-0.1
- added M5: Module-knock-0.2, hellen-one-knock-0.2:knock, symbol hellen-one-knock-0.2:Module-knock-0.2
- added M8: Module-power_12and5V-0.1, hellen-one-power_12and5V-0.1:power_12and5V, symbol power_12and5V-0.1:Module-power_12and5V-0.1
- added M9: Module-wbo-0.5, hellen-one-wbo-0.5:wbo, symbol hellen-one-wbo-0.5:Module-wbo-0.5
Connections:
- net +12V: now also M8.E2 (V12)
- net +12V_PROT: now also M8.E5 (EN_5VP)
- net +12V_RAW: now also M8.V3 (V12_RAW)
- net +3V3: now also M3.N29 (V33)
- net +5V: now also M11.E4 (V5_IN), M3.N28 (VCC), M8.E4 (V5), M9.W1 (V5_IN)
- net +5VA: now also M3.W0 (V5A), M5.E1 (V5A)
- net +5VP: now also M8.V4 (5VP)
- net +ETB: now also M3.E17 (OUT_PWM2)
- net -ETB: now also M3.E16 (OUT_PWM3)
- net CAN+: now also M3.W9 (CANH), M9.W4 (CANH)
- net CAN-: now also M3.W10 (CANL), M9.W3 (CANL)
- net CHECK_ENGINE: now also M3.E22 (OUT_IO8)
- net ETB_EN: now also M3.E13 (OUT_IO12)
- net FUEL_CONSUM: now also M3.E25 (OUT_PWM7)
- net FUEL_PUMP_RELAY: now also M3.E8 (OUT_IO1)
- net GND: now also M11.G (GND), M3.G (GND), M5.E2 (GND), M8.S1 (GND), M9.E6 (LSU_H-), M9.G (GND)
- net GNDA: now also M3.W (GNDA)
- net IDLE: now also M3.E21 (OUT_IO4)
- net IGN1: now also M3.W8 (IGN1)
- net IGN2: now also M3.W7 (IGN2)
- net IGN3: now also M3.W6 (IGN3)
- net IGN4: now also M3.W5 (IGN4)
- net IGN5: now also M3.W4 (IGN5)
- net IGN6: now also M3.W3 (IGN6)
- net IGN7: now also M3.W2 (IGN7)
- net IGN8: now also M3.W1 (IGN8)
- net INJ1: now also M3.E19 (OUT_INJ1)
- net INJ2: now also M3.E18 (OUT_INJ2)
- net INJ3: now also M3.E29 (OUT_INJ3)
- net INJ4: now also M3.E30 (OUT_INJ4)
- net INJ5: now also M3.E31 (OUT_INJ5)
- net INJ6: now also M3.E32 (OUT_INJ6)
- net INJ7: now also M3.E33 (OUT_INJ7)
- net INJ8: now also M3.E34 (OUT_INJ8)
- net IN_A1: now also M3.S15 (IN_O2S2)
- net IN_A2: now also M3.S19 (IN_MAP3)
- net IN_A3: now also M3.S11 (IN_AUX3)
- net IN_A4: now also M3.S18 (IN_RES3)
- net IN_AFR: now also M3.S16 (IN_O2S)
- net IN_CAM1: now also M3.S24 (IN_CAM)
- net IN_CAM2: now also M3.S10 (IN_AUX4)
- net IN_CLT: now also M3.S28 (IN_CLT)
- net IN_CRANK: now also M11.E3 (OUT), M3.S22 (IN_CRANK)
- net IN_CRANK+: now also M11.W2 (VR+)
- net IN_CRANK-: now also M11.W1 (VR-)
- net IN_D1: now also M3.S4 (IN_D1)
- net IN_D2: now also M3.S3 (IN_D2)
- net IN_D3: now also M3.S2 (IN_D3)
- net IN_D4: now also M3.S1 (IN_D4)
- net IN_IAT: now also M3.S26 (IN_IAT)
- net IN_KNOCK1: now also M3.S23 (IN_KNOCK), M5.E3 (OUT_KNOCK)
- net IN_KNOCK1_RAW: now also M5.W1 (IN_KNOCK)
- net IN_MAF: now also M3.S21 (IN_MAP1)
- net IN_MAP2: now also M3.S20 (IN_MAP2)
- net IN_PPS1: now also M3.S31 (IN_PPS)
- net IN_PPS2: now also M3.S12 (IN_AUX2)
- net IN_RES1: now also M3.S17 (IN_RES1)
- net IN_RES2: now also M3.S14 (IN_RES2)
- net IN_TPS1: now also M3.S30 (IN_TPS)
- net IN_TPS2: now also M3.S13 (IN_AUX1)
- net IN_VIGN: now also M8.V2 (IN_VIGN)
- net IN_VSS: now also M3.S25 (IN_VSS)
- net LSU_CALIBR_RES: now also M9.E4 (LSU_Rtrim)
- net LSU_HEAT-: now also M9.E5 (LSU_H+)
- net LSU_PUMP_I: now also M9.E3 (LSU_Ip)
- net LSU_SENSOR_U: now also M9.E1 (LSU_Un)
- net LSU_SENSOR_U/PUMP_I: now also M9.E2 (LSU_Vm)
- net MAIN_RELAY: now also M3.E6 (OUT_IO3)
- net OUT1: now also M3.E7 (OUT_IO5)
- net OUT2: now also M3.E9 (OUT_IO6)
- net OUT3: now also M3.E28 (OUT_PWM8)
- net RX1: now also M3.N24 (UART8_RX)
- net RX2: now also M3.N18 (UART2_RX)
- net SPI3_CS: now also M3.N10 (SPI3_CS)
- net SPI3_MISO: now also M3.N12 (SPI3_MISO)
- net SPI3_MOSI: now also M3.N13 (SPI3_MOSI)
- net SPI3_SCK: now also M3.N11 (SPI3_SCK)
- net TACH: now also M3.E27 (OUT_PWM1)
- net THRESHOLD_VR: now also M11.E1 (Thresh_IN), M3.E26 (OUT_PWM6)
- net TX1: now also M3.N25 (UART8_TX)
- net TX2: now also M3.N17 (UART2_TX)
- net USBM: now also M3.N2 (USBM)
- net USBP: now also M3.N3 (USBP)
- net V12_PERM: now also M8.V1 (V12_PERM)
- net VBAT: now also M3.N27 (VBAT), M8.E1 (VBAT)
- net VBUS: now also M3.N4 (VBUS)
- net VIGN: now also M3.N26 (IN_VIGN), M8.E3 (VIGN)
- net VREF2: now also M5.W2 (VREF)
- net VR_ANALOG: now also M11.E2 (OUT_A), M3.S9 (IN_SENS1)
- net VVT1_1: now also M3.E10 (OUT_IO10)
- net VVT1_2: now also M3.E23 (OUT_IO7)
- net VVT2_B1: now also M3.E14 (OUT_PWM5)
- net VVT2_B2: now also M3.E15 (OUT_PWM4)
- net WASTEGATE: now also M3.E12 (OUT_IO2)
- net at J8.5 (Pin_5): now also M9.W5 (nReset)
- net at J8.4 (Pin_4): now also M9.W6 (SWDIO)
- net at J8.2 (Pin_2): now also M9.W7 (SWCLK)
- net at J8.1 (Pin_1): now also M9.W8 (V33_OUT)
- new net: M9.J2 (SEL2), M9.J_VCC2 (PULL_UP2)
- no-connect marks 62 -> 72
Other:
- note removed: "Baro"
- note removed: "C540240"
- note removed: "C540241"
- note removed: "C540242"
- note removed: "C540243"
- note removed: "Protected 5V analog power supply"
- note removed: "SOIC-8"
- note removed: "TSON-10"
- moved on the sheet: BT1, D9, J1, M4D, P15, P16, P2, P3, P4, P5, R23, R6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

Commit message: SD&accel
Parts:
- removed M4: Module-input-0.1, hellen-one-input-0.1:input, symbol hellen-one-input-0.1:Module-input-0.1
- removed R6, R7: 2.7k, hellen-one-common:R0603, symbol hellen-one-common:Res
Connections:
- no-connect marks 72 -> 70
Other:
- note removed: "Without accelerometer and SD card"
- moved on the sheet: P15, P16
