File: hellen121vag_rev_c.kicad_sch (KiCad schematic)
At the start: 122 parts, among them J1 USB_B_Mini, J10 AudioJack_THR, J2 Conn_01x01, J3 Conn_01x01, J4 Conn_01x01, J5 Conn_01x01, J6 Conn_01x01, J7 Conn_01x08, J8 Conn_01x06, M1 Module-can-0.1, M10 Module-can-0.1, M11 Module-vr-0.1, M12 Module-dinput4-0.1, M2 Module-power5-0.2, M3 Module-mcu-0.2, M4 Module-input-0.1, M5 Module-knock-0.1, M6 Module-output-0.2, M7 Module-ign8-0.1, M8 Module-power12-0.2, M9 Module-wbo-0.1, P1 368255-2, P10 Pad, P11 Pad, P12 Pad, P13 Pad, P14 Pad, P17 Pad, P2 Pad, P20 Pad, P28 Pad, P3 Pad, P4 Pad, P40 Pad, P41 Pad, P43 Pad, P44 Pad, P45 Pad, P46 Pad, P48 Pad, P49 Pad, P5 Pad, P56 Pad, P6 Pad, P61 Pad, P63 Pad, P64 Pad, P66 Pad, P67 Pad, P68 Pad, P69 Pad, P7 Pad, P74 Pad, P8 Pad, P80 Pad, P9 Pad, U1 L6205PD, U2 LPS25HB, U3 MCP6002-xSN

Commit message: Rev. b is fixed rev. a
Parts:
- removed J7: Conn_01x08, Connector_PinHeader_2.54mm:PinHeader_1x08_P2.54mm_Vertical, symbol Connector_Generic:Conn_01x08
- removed P10, P11, P12, P13, P14, P17, P20, P28, P40, P41, P43, P44, P45, P46, P48, P49, P5, P56, P6, P61, P63, P64, P66, P67, P68, P69, P7, P74, P8, P80, P9: Pad, hellen-one-common:PAD-TH, symbol hellen-one-common:Pad
- added C18: 100n, hellen-one-common:C0603, symbol hellen-one-common:Cap
- added J11: Conn_01x06, Connector_PinHeader_2.54mm:PinHeader_1x06_P2.54mm_Vertical, symbol Connector_Generic:Conn_01x06
- added J7, J9: Conn_01x04, Connector_PinHeader_2.54mm:PinHeader_1x04_P2.54mm_Vertical, symbol Connector_Generic:Conn_01x04
- added M13: Module-sd-0.1, hellen-one-sd-0.1:sd, symbol hellen-one-sd-0.1:Module-sd-0.1
- added U4: LIS2DW12TR, hellen-one-common:LGA-12_2x2mm_P0.5mm, symbol hellen-one-common:LIS2DW12TR
- added V10, V11, V12, V13, V14, V17, V20, V28, V40, V41, V43, V44, V45, V46, V48, V49, V56, V61, V63, V64, V66, V67, V68, V69, V74, V80, V9, VIN1, VIN2, VIN3, VIN4, VOUT1, VOUT2, VOUT3: Pad, hellen-one-common:PAD-TH, symbol hellen-one-common:Pad
- F1: LCSC (none) -> C182446; MyComment DNP -> (none)
Connections:
- net +12V: now also J2.1 (Pin_1)
- net +12V_PROT: now also D10.1 (K), D11.1 (K), D12.1 (K)
- net +12V_RAW: no longer D10.1 (K), D11.1 (K), D12.1 (K), J2.1 (Pin_1)
- net +3V3: now also C18.2, J11.1 (Pin_1), M13.V1 (V33), U4.10 (Vdd_IO), U4.9 (Vdd)
- net CAM1: now also P3.1 (Pin_1)
- net CAM2: now also P4.1 (Pin_1)
- net CRANK: now also P2.1 (Pin_1)
- net GND: now also C18.1, J11.6 (Pin_6), M13.G (GND), M13.V2 (GND), M13.V3 (GND), U4.6 (GND), U4.7 (RES), U4.8 (GND)
- net IN_A1: now also VIN1.1 (Pin_1); no longer P2.1 (Pin_1)
- net IN_A2: now also VIN2.1 (Pin_1); no longer P4.1 (Pin_1)
- net IN_A3: now also VIN3.1 (Pin_1)
- net IN_A4: now also VIN4.1 (Pin_1); no longer P3.1 (Pin_1)
- net IN_AFR: now also V14.1 (Pin_1)
- net RX1: now also J7.3 (Pin_3)
- net RX2: now also J7.1 (Pin_1)
- net SPI3_CS: now also J9.4 (Pin_4)
- net SPI3_MISO: now also J9.2 (Pin_2)
- net SPI3_MOSI: now also J9.1 (Pin_1)
- net SPI3_SCK: now also J9.3 (Pin_3)
- net TX1: now also J7.4 (Pin_4)
- net TX2: now also J7.2 (Pin_2)
- net at P1.10: now also V10.1 (Pin_1)
- net at P1.11: now also V11.1 (Pin_1)
- net at P1.12: now also V12.1 (Pin_1)
- net at P1.13: now also V13.1 (Pin_1)
- net at P1.17: now also V17.1 (Pin_1)
- net at P1.20: now also V20.1 (Pin_1)
- net at P1.28: now also V28.1 (Pin_1)
- net at P1.40: now also V40.1 (Pin_1)
- net at P1.41: now also V41.1 (Pin_1)
- net at P1.43: now also V43.1 (Pin_1)
- net at P1.44: now also V44.1 (Pin_1)
- net at P1.45: now also V45.1 (Pin_1)
- net at P1.46: now also V46.1 (Pin_1)
- net at P1.48: now also V48.1 (Pin_1)
- net at P1.49: now also V49.1 (Pin_1)
- net at P1.56: now also V56.1 (Pin_1)
- net at P1.61: now also V61.1 (Pin_1)
- net at P1.63: now also V63.1 (Pin_1)
- net at P1.64: now also V64.1 (Pin_1)
- net at P1.66: now also V66.1 (Pin_1)
- net at P1.67: now also V67.1 (Pin_1)
- net at P1.68: now also V68.1 (Pin_1)
- net at P1.69: now also V69.1 (Pin_1)
- net at P1.74: now also V74.1 (Pin_1)
- net at P1.80: now also V80.1 (Pin_1)
- net at P1.9: now also V9.1 (Pin_1)
- net at M6.W9 (OUT_LOW7_PULLUP): now also VOUT1.1 (Pin_1)
- net SPI1_SCK: now reaches M3.E1 (SPI1_SCK)
- net SPI1_SCK: now also U4.1 (SCL/SPC)
- net SPI1_MISO: now reaches M3.E2 (SPI1_MISO)
- net SPI1_MISO: now also U4.3 (SA0/SDO)
- net SPI1_MOSI: now reaches M3.E3 (SPI1_MOSI)
- net SPI1_MOSI: now also U4.4 (SDA/SDI)
- net SPI1_CS: now reaches M3.E4 (SPI1_CS1)
- net SPI1_CS: now also U4.2 (~CS)
- net SD_SCK: now reaches M3.N20 (SPI2_SCK)
- net SD_SCK: now also J11.4 (Pin_4), M13.V6 (SD_SCK)
- net SD_MISO: now reaches M3.N21 (SPI2_MISO)
- net SD_MISO: now also J11.5 (Pin_5), M13.V7 (SD_MISO)
- net SD_MOSI: now reaches M3.N22 (SPI2_MOSI)
- net SD_MOSI: now also J11.3 (Pin_3), M13.V5 (SD_MOSI)
- net SD_CS: now reaches M3.N23 (SPI2_CS)
- net SD_CS: now also J11.2 (Pin_2), M13.V4 (SD_CS)
- net at M6.S12 (OUT_LOW8_PULLUP): now also VOUT2.1 (Pin_1)
- net at M6.S8 (OUT_LOW1): now also VOUT3.1 (Pin_1)
- no-connect marks 67 -> 62
Other:
- note added: "Accelerometer"
- note removed: "Without accelerometer and SD card"
